File: X610.kicad_pcb (KiCad board)
At the start: 8 copper layers, 33 x 44 mm, 103 parts, among them J1 Conn_01x02, J2 MR30, J3 PA, J4 Conn_01x01, J5 Conn_01x01, J6 PA, J7 Conn_01x06, J8 PA, J9 GH, SW1 SW_Push, SW2 SW_Push, U1 STM32G431CBUx, U2 DRV8328C, U3 TCAN857-Q1, U4 LMR516xx, U5 NJM2884, U6 CH213K, Y1 25MHz

Commit message: 2回目の発注
Parts:
- removed H1: MountingHole, MountingHole:MountingHole_3.2mm_M3
- added D6: SS2040FL, Diode_SMD:D_SOD-123, B.Cu at (157.0, 98.2)
- added D7: D_Zener, Diode_SMD:D_SOD-323, B.Cu at (169.8, 88.0)
- added D8: D_Zener, Diode_SMD:D_SOD-323, B.Cu at (164.6, 88.0)
- added D9: D_Zener, Diode_SMD:D_SOD-323, B.Cu at (159.4, 88.0)
- R12, R16, R19: value 22k -> 2.2k
- R14, R17, R20: value 10 -> 1k
- R21, R22, R23, R24, R25, R26: value 100 -> 47
- moved J1 2.04 mm to (153.1, 117.1)
- moved J3 0.81 mm to (151.1, 113.0)
Connections:
- C19 pad 1: +24V -> Net-(D6-K)
- U1 pad 12: unconnected-(U1-PA4-Pad12) -> /DRIVER/nSLEEP
- U4 pad 5: +24V -> Net-(D6-K)
Routing:
- net /DRIVER/nSLEEP: track 6.40 -> 18.7 mm, vias 0 -> 2
- net Net-(D8-K): track 0.88 -> 3.09 mm
- net Net-(D7-K): track 0.88 -> 3.09 mm
- net Net-(D9-K): track 0.88 -> 3.09 mm
- net Net-(D6-K): track 0.00 -> 2.13 mm, vias 0 -> 1
- net /MCU/LIMIT_SW: track 12.3 -> 14.0 mm
- net /CANFD/CANFD_P: track 3.28 -> 4.26 mm
- net Net-(J1-Pin_1): track 3.95 -> 4.68 mm
- net GND: vias 157 -> 160
Other:
- board text added: "X610 v1.1.0"
- board text removed: "G"
- board text removed: "V"
- board text removed: "X610 v1.0.0"
