File: driver.kicad_sch (KiCad schematic)
At the start: 34 parts, among them J2 MR30, U2 DRV8328C

Commit message: 2回目の発注
Parts:
- added D7, D8, D9: D_Zener, Diode_SMD:D_SOD-323, symbol Device:D_Zener
- R12, R16, R19: value 22k -> 2.2k
- R14, R17, R20: value 10 -> 1k
- R21, R22, R23, R24, R25, R26: value 100 -> 47
Connections:
- net GND: now also D7.2 (A), D8.2 (A), D9.2 (A)
- net at Q1.9 (G2), R22.2: now also D9.1 (K)
- net at Q2.9 (G2), R24.2: now also D8.1 (K)
- net at Q3.9 (G2), R26.2: now also D7.1 (K)
