File: mcu.kicad_sch (KiCad schematic)
At the start: 22 parts, among them J1 Conn_01x02, SW1 SW_Push, SW2 SW_Push, U1 STM32G431CBUx, Y1 25MHz

Commit message: 2回目の発注
Connections:
- net nSLEEP: now reaches U1.12 (PA4)
Changed lines of the file:
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@@
+	(wire
+		(pts
+			(xy 175.26 77.47) (xy 177.8 77.47)
+		)
+		(stroke
+			(width 0)
+			(type default)
+		)
+	)
 	(wire
 		(pts
@@
 		(effects
 			(font
+				(size 1.27 1.27)
+			)
+			(justify left)
+		)
+	)
+	(hierarchical_label "nSLEEP"
+		(shape output)
+		(at 177.8 77.47 0)
+		(effects
+			(font
