File: power.kicad_sch (KiCad schematic)
At the start: 20 parts, among them J4 Conn_01x01, J5 Conn_01x01, U4 LMR516xx, U5 NJM2884

Commit message: 2回目の発注
Parts:
- added D6: SS2040FL, Diode_SMD:D_SOD-123, symbol Device:D
Connections:
- net +24V: now also D6.2 (A); no longer C19.1, U4.5 (VIN)
- new net: C19.1, D6.1 (K), U4.5 (VIN)
Changed lines of the file:
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@@
+	)
+	(junction
+		(at 77.47 97.79)
+		(diameter 0)
+		(color 0 0 0 0)
 	)
 	(junction
@@
 	)
 	(junction
-		(at 77.47 97.79)
-		(diameter 0)
-		(color 0 0 0 0)
-	)
-	(junction
 		(at 85.09 66.04)
 		(diameter 0)
@@
 	(wire
 		(pts
+			(xy 226.06 129.54) (xy 229.87 129.54)
+		)
+		(stroke
+			(width 0)
+			(type default)
+		)
+	)
+	(wire
+		(pts
+			(xy 140.97 100.33) (xy 140.97 101.6)
+		)
+		(stroke
+			(width 0)
+			(type default)
+		)
+	)
+	(wire
+		(pts
 			(xy 77.47 97.79) (xy 107.95 97.79)
-		)
-		(stroke
-			(width 0)
-			(type default)
-		)
-	)
-	(wire
-		(pts
-			(xy 226.06 129.54) (xy 229.87 129.54)
-		)
-		(stroke
-			(width 0)
-			(type default)
-		)
-	)
-	(wire
-		(pts
-			(xy 140.97 100.33) (xy 140.97 101.6)
 		)
 		(stroke
@@
 	)
 	(symbol
+		(lib_id "Device:D")
+		(at 73.66 97.79 180)
+		(unit 1)
+		(exclude_from_sim no)
+		(in_bom yes)
+		(on_board yes)
+		(dnp no)
+		(fields_autoplaced yes)
+		(property "Reference" "D6"
+			(at 73.66 91.44 0)
+			(effects
+				(font
+					(size 1.27 1.27)
+				)
+			)
+		)
+		(property "Value" "SS2040FL"
+			(at 73.66 93.98 0)
+			(effects
+				(font
+					(size 1.27 1.27)
+				)
+			)
+		)
+		(property "Footprint" "Diode_SMD:D_SOD-123"
+			(at 73.66 97.79 0)
+			(effects
+				(font
+					(size 1.27 1.27)
+				)
+				(hide yes)
+			)
+		)
+		(property "Datasheet" "~"
+			(at 73.66 97.79 0)
+			(effects
+				(font
+					(size 1.27 1.27)
+				)
+				(hide yes)
+			)
+		)
+		(property "Description" "Diode"
+			(at 73.66 97.79 0)
+			(effects
+				(font
+					(size 1.27 1.27)
+				)
+				(hide yes)
+			)
+		)
+		(property "Sim.Device" "D"
+			(at 73.66 97.79 0)
+			(effects
+				(font
+					(size 1.27 1.27)
+				)
+				(hide yes)
+			)
+		)
+		(property "Sim.Pins" "1=K 2=A"
+			(at 73.66 97.79 0)
+			(effects
+				(font
+					(size 1.27 1.27)
+				)
+				(hide yes)
+			)
+		)
+		(pin "1"
+		)
+		(pin "2"
+		)
+		(instances
+			(project "X610"
+				(path "/73db8ec9-de03-4da6-b9c5-ef3a35d8ec71/faf9e788-172d-4cd9-859c-c7d01e0fab01"
+					(reference "D6")
+					(unit 1)
+				)
+			)
+		)
+	)
+	(symbol
 		(lib_id "power:GND")
 		(at 189.23 109.22 0)
@@
 	(symbol
 		(lib_id "power:+12V")
-		(at 77.47 97.79 0)
+		(at 69.85 97.79 90)
 		(unit 1)
 		(exclude_from_sim no)
@@
 		(dnp no)
 		(property "Reference" "#PWR060"
-			(at 77.47 101.6 0)
+			(at 73.66 97.79 0)
 			(effects
 				(font
@@
 		)
 		(property "Value" "+24V"
-			(at 74.93 93.726 0)
+			(at 65.786 100.33 0)
 			(effects
 				(font
@@
 		)
 		(property "Footprint" ""
-			(at 77.47 97.79 0)
+			(at 69.85 97.79 0)
 			(effects
 				(font
@@
 		)
 		(property "Datasheet" ""
-			(at 77.47 97.79 0)
+			(at 69.85 97.79 0)
 			(effects
 				(font
@@
 		)
 		(property "Description" "Power symbol creates a global label with name \"+12V\""
-			(at 77.47 97.79 0)
-			(effects
-				(font
+			(at 69.85 97.79 0)
+			(effects
+				(font
